File: main_board.brd (EAGLE design)
At the start: 123.2 x 81 mm, 46 parts, among them P1 ST-TF-003A, U1 STM32F407VGT6, U2 USBLC6-2, U3 MCP1700T-3302E, U4 LTC4054LES5-4.2#TRPBF, X1 MicroUSB-B

Commit message: pcb in progress..
Routing:
- net GND: track 301.9 -> 308.1 mm
- net VDD: track 304.6 -> 305.1 mm
Changed lines of the file:
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@@
 <wire x1="58.1" y1="58.42" x2="58.1" y2="60.96" width="0.8128" layer="1"/>
 <wire x1="58.1" y1="60.96" x2="58.608" y2="61.468" width="0.8128" layer="1"/>
-<wire x1="69.088" y1="61.468" x2="58.608" y2="61.468" width="0.8128" layer="1"/>
+<wire x1="69.088" y1="61.468" x2="68.58" y2="61.468" width="0.8128" layer="1"/>
+<wire x1="68.58" y1="61.468" x2="58.608" y2="61.468" width="0.8128" layer="1"/>
 <wire x1="45.72" y1="73.66" x2="53.34" y2="73.66" width="0.8128" layer="1"/>
 <wire x1="53.34" y1="73.66" x2="58.42" y2="68.58" width="0.8128" layer="1"/>
@@
 <wire x1="72.914" y1="64.135" x2="71.755" y2="64.135" width="0.8128" layer="1"/>
 <wire x1="71.755" y1="64.135" x2="71.12" y2="63.5" width="0.8128" layer="1"/>
-<wire x1="71.12" y1="63.5" x2="68.8975" y2="61.2775" width="0.8128" layer="1"/>
+<wire x1="68.8975" y1="61.2775" x2="71.12" y2="63.5" width="0.8128" layer="1"/>
 <wire x1="83.82" y1="30.48" x2="76.2" y2="38.1" width="0.8128" layer="1"/>
 <wire x1="76.2" y1="38.1" x2="71.12" y2="38.1" width="0.8128" layer="1"/>
@@
 <wire x1="144.53" y1="31.97" x2="141.7" y2="31.97" width="0.3" layer="1"/>
 <wire x1="141.7" y1="31.97" x2="141.539" y2="32.131" width="0.3" layer="1"/>
-<wire x1="144.53" y1="31.97" x2="147.54" y2="31.97" width="0.6096" layer="1"/>
-<wire x1="147.54" y1="31.97" x2="149.86" y2="34.29" width="0.6096" layer="1"/>
-<wire x1="149.86" y1="34.29" x2="149.86" y2="45.72" width="0.6096" layer="1"/>
+<wire x1="144.53" y1="31.97" x2="147.8067" y2="31.97" width="0.6096" layer="1"/>
+<wire x1="147.8067" y1="31.97" x2="149.86" y2="34.0233" width="0.6096" layer="1"/>
+<wire x1="149.86" y1="34.0233" x2="149.86" y2="45.72" width="0.6096" layer="1"/>
 <wire x1="149.86" y1="45.72" x2="147" y2="48.58" width="1.016" layer="1"/>
 <wire x1="147" y1="48.58" x2="143.51" y2="48.58" width="1.016" layer="1"/>
@@
 <wire x1="77.41" y1="58.34" x2="76.28" y2="58.34" width="0.3" layer="1"/>
 <wire x1="76.28" y1="58.34" x2="71.12" y2="63.5" width="0.3" layer="1"/>
-<wire x1="69.088" y1="61.468" x2="68.8975" y2="61.2775" width="0" layer="19" extent="1-1"/>
+<wire x1="68.58" y1="61.468" x2="68.707" y2="61.468" width="0.3" layer="1"/>
+<wire x1="68.707" y1="61.468" x2="68.8975" y2="61.2775" width="0.3" layer="1"/>
 </signal>
 <signal name="GND" class="1">
@@
 <wire x1="142.24" y1="42.76" x2="142.24" y2="43.18" width="0.3" layer="1"/>
 <via x="142.24" y="43.18" extent="1-16" drill="1"/>
-<wire x1="145.13" y1="25.17" x2="154.63" y2="25.17" width="0" layer="19" extent="1-1"/>
+<wire x1="154.63" y1="25.17" x2="148.36" y2="25.17" width="0.3" layer="1"/>
 </signal>
 <signal name="I2C_SDA">
@@
 <contactref element="C1" pad="2"/>
 <wire x1="85.59" y1="61.02" x2="85.59" y2="68.191" width="0.3" layer="1"/>
-<wire x1="85.59" y1="68.191" x2="86.614" y2="69.215" width="0.3" layer="1"/>
-<wire x1="86.614" y1="69.215" x2="86.614" y2="70.866" width="0.3" layer="1"/>
+<wire x1="86.614" y1="69.215" x2="85.59" y2="68.191" width="0.3" layer="1"/>
 <wire x1="91.76" y1="71.12" x2="86.614" y2="71.12" width="0.8128" layer="1"/>
-<wire x1="86.614" y1="71.12" x2="86.36" y2="71.374" width="0.3" layer="1"/>
-<wire x1="86.614" y1="70.866" x2="86.36" y2="71.374" width="0" layer="19" extent="1-1"/>
+<wire x1="86.36" y1="71.374" x2="86.614" y2="71.12" width="0.3" layer="1"/>
+<wire x1="86.614" y1="71.12" x2="86.614" y2="69.215" width="0.3" layer="1"/>
 </signal>
 <signal name="N$2">
@@
 <via x="138.557" y="38.227" extent="1-16" drill="0.9"/>
 <wire x1="138.557" y1="38.227" x2="141.224" y2="35.56" width="0.3" layer="1"/>
-<wire x1="141.224" y1="35.56" x2="144.78" y2="35.56" width="0.3" layer="1"/>
-<wire x1="144.78" y1="35.56" x2="144.53" y2="35.27" width="0" layer="19" extent="1-1"/>
+<wire x1="144.78" y1="35.56" x2="141.224" y2="35.56" width="0.3" layer="1"/>
+<wire x1="144.53" y1="35.27" x2="144.53" y2="35.31" width="0.3" layer="1"/>
+<wire x1="144.53" y1="35.31" x2="144.78" y2="35.56" width="0.3" layer="1"/>
 </signal>
 <signal name="SD_DAT3">
@@
 <mfgpreviewcolor name="substratecolor" color="0xFF786E46"/>
 </mfgpreviewcolors>
+<errors>
+</errors>
 </board>
 </drawing>

Commit message: pcb almost done
Parts:
- moved C21 66.6 mm to (77.9, 62.3)
- moved R5 66.6 mm to (73.2, 63.1)
- moved R7 66.6 mm to (69.6, 59.9)
- moved U2 66.6 mm to (86.3, 58.2)
- moved U4 66.6 mm to (74.9, 59.5)
- moved LED1 66.6 mm to (71.0, 54.4)
- moved R6 66.6 mm to (71.0, 57.0)
- moved X1 66.6 mm to (95.2, 58.2)
- moved C22 65.9 mm to (78.4, 10.5)
- moved P1 63.5 mm to (90.2, 10.2)
- moved R9 60.9 mm to (79.9, 53.2), turned to 180 degrees
- moved JP3 58.7 mm to (67.0, 66.9), turned to 0 degrees
- moved R8 57.9 mm to (91.4, 24.1)
- moved S2 56.3 mm to (87.6, 31.8)
- moved R10 54.5 mm to (84.8, 53.2), turned to 180 degrees
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Routing:
- net VDD: track 305.1 -> 281.8 mm
- net SD_CMD: track 68.0 -> 45.1 mm
- net SD_DAT2: track 57.8 -> 38.7 mm
- net SD_CLK: track 59.7 -> 40.8 mm
- net VBAT+: track 58.3 -> 39.7 mm
- net SD_DAT3: track 57.8 -> 41.5 mm
- net SD_DAT0: track 76.7 -> 61.7 mm
- net SD_DAT1: track 73.6 -> 59.2 mm
- net D-_INT: track 85.4 -> 73.9 mm
- net D+_PROT: track 89.0 -> 78.2 mm
- net NCHRG: track 58.1 -> 48.3 mm
- net BTN_0: track 65.0 -> 57.3 mm
- net I2C_SCL: track 84.5 -> 91.8 mm
- net BTN_2: track 53.0 -> 46.6 mm
- net BTN_4: track 53.1 -> 46.7 mm
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Other:
- board size 123.2 x 81 mm -> 100.3 x 69.8 mm

Commit message: pcb almost done
Parts:
- flipped S1 to the top, turned to 180 degrees
Routing:
- net N$7: track 17.2 -> 20.0 mm
Changed lines of the file:
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@@
 <layer number="23" name="tOrigins" color="15" fill="1" visible="yes" active="yes"/>
 <layer number="24" name="bOrigins" color="15" fill="1" visible="yes" active="yes"/>
-<layer number="25" name="tNames" color="7" fill="1" visible="yes" active="yes"/>
-<layer number="26" name="bNames" color="7" fill="1" visible="yes" active="yes"/>
+<layer number="25" name="tNames" color="7" fill="1" visible="no" active="yes"/>
+<layer number="26" name="bNames" color="7" fill="1" visible="no" active="yes"/>
 <layer number="27" name="tValues" color="7" fill="1" visible="no" active="yes"/>
 <layer number="28" name="bValues" color="7" fill="1" visible="no" active="yes"/>
@@
 <attribute name="VALUE" x="80.5688" y="55.7022" size="1.27" layer="27" rot="R180"/>
 </element>
-<element name="S1" library="SSA12G" package="SW_SSA12G" value="" x="46.101" y="67.945" smashed="yes" rot="MR0">
-<attribute name="AVAILABILITY" value="In Stock" x="9.271" y="22.225" size="1.778" layer="28" rot="MR0" display="off"/>
-<attribute name="COMMENT" value="1-1437575-5" x="9.271" y="22.225" size="1.778" layer="28" rot="MR0" display="off"/>
-<attribute name="DESCRIPTION" value=" 2 Position SPDT Extended Top Actuator Through Hole Vertical Mount Slide Switch " x="9.271" y="22.225" size="1.778" layer="28" rot="MR0" display="off"/>
-<attribute name="MF" value="TE Connectivity" x="9.271" y="22.225" size="1.778" layer="28" rot="MR0" display="off"/>
-<attribute name="MP" value="SSA12G" x="9.271" y="22.225" size="1.778" layer="28" rot="MR0" display="off"/>
-<attribute name="NAME" x="50.854090625" y="70.196459375" size="1.779159375" layer="26" rot="MR0"/>
-<attribute name="PACKAGE" value="None" x="9.271" y="22.225" size="1.778" layer="28" rot="MR0" display="off"/>
-<attribute name="PRICE" value="None" x="9.271" y="22.225" size="1.778" layer="28" rot="MR0" display="off"/>
-<attribute name="VALUE" x="50.855709375" y="63.94103125" size="1.779759375" layer="28" rot="MR0"/>
+<element name="S1" library="SSA12G" package="SW_SSA12G" value="" x="46.0883" y="67.9069" smashed="yes" rot="R180">
+<attribute name="AVAILABILITY" value="In Stock" x="9.2583" y="113.6269" size="1.778" layer="27" rot="R180" display="off"/>
+<attribute name="COMMENT" value="1-1437575-5" x="9.2583" y="113.6269" size="1.778" layer="27" rot="R180" display="off"/>
+<attribute name="DESCRIPTION" value=" 2 Position SPDT Extended Top Actuator Through Hole Vertical Mount Slide Switch " x="9.2583" y="113.6269" size="1.778" layer="27" rot="R180" display="off"/>
+<attribute name="MF" value="TE Connectivity" x="9.2583" y="113.6269" size="1.778" layer="27" rot="R180" display="off"/>
+<attribute name="MP" value="SSA12G" x="9.2583" y="113.6269" size="1.778" layer="27" rot="R180" display="off"/>
+<attribute name="NAME" x="50.841390625" y="65.655440625" size="1.779159375" layer="25" rot="R180"/>
+<attribute name="PACKAGE" value="None" x="9.2583" y="113.6269" size="1.778" layer="27" rot="R180" display="off"/>
+<attribute name="PRICE" value="None" x="9.2583" y="113.6269" size="1.778" layer="27" rot="R180" display="off"/>
+<attribute name="VALUE" x="50.843009375" y="71.91086875" size="1.779759375" layer="27" rot="R180"/>
 </element>
 <element name="S2" library="int-1500m90b" package="SW6-3.25-10X10X8.6MM" value="INT-1500M90B" x="87.63" y="31.75" smashed="yes">
@@
 <wire x1="68.3641" y1="63.8048" x2="63.5" y2="63.8048" width="1.016" layer="1"/>
 <wire x1="63.5" y1="63.8048" x2="63.1825" y2="63.8048" width="1.016" layer="1"/>
-<wire x1="48.601" y1="67.945" x2="49.871" y2="66.675" width="1.016" layer="1"/>
-<wire x1="49.871" y1="66.675" x2="49.871" y2="65.699" width="1.016" layer="1"/>
 <wire x1="51.5817" y1="63.9883" x2="63.9699" y2="63.9883" width="1.016" layer="1"/>
-<wire x1="49.871" y1="65.699" x2="51.5817" y2="63.9883" width="1.016" layer="1"/>
+<wire x1="51.5817" y1="63.9883" x2="49.871" y2="65.699" width="1.016" layer="1"/>
 <wire x1="63.9699" y1="63.9883" x2="63.9699" y2="65.1383" width="1.016" layer="1"/>
 <wire x1="63.9699" y1="65.1383" x2="65.7098" y2="66.8782" width="1.016" layer="1"/>
 <wire x1="63.9699" y1="63.9883" x2="63.7864" y2="63.8048" width="0.3" layer="1"/>
 <wire x1="63.7864" y1="63.8048" x2="63.5" y2="63.8048" width="0.3" layer="1"/>
+<wire x1="49.871" y1="65.699" x2="48.5883" y2="66.9817" width="1.016" layer="1"/>
+<wire x1="48.5883" y1="66.9817" x2="48.5883" y2="67.9069" width="1.016" layer="1"/>
 </signal>
 <signal name="VDDA" class="1">
@@
 <wire x1="58.928" y1="60.409" x2="55.141" y2="60.409" width="0.8128" layer="1"/>
 <wire x1="55.141" y1="60.409" x2="54.991" y2="60.259" width="0.3" layer="1"/>
-<wire x1="54.991" y1="60.259" x2="51.882" y2="60.259" width="1.016" layer="1"/>
-<wire x1="51.882" y1="60.259" x2="46.0502" y2="66.0908" width="1.016" layer="1"/>
-<wire x1="46.101" y1="67.945" x2="46.0502" y2="67.8942" width="1.016" layer="1"/>
-<wire x1="46.0502" y1="67.8942" x2="46.0502" y2="66.0908" width="1.016" layer="1"/>
+<wire x1="54.991" y1="60.259" x2="52.07" y2="60.259" width="1.016" layer="1"/>
+<wire x1="52.07" y1="60.259" x2="51.882" y2="60.259" width="1.016" layer="1"/>
+<wire x1="51.882" y1="60.259" x2="47.056" y2="60.259" width="1.016" layer="1"/>
+<wire x1="47.056" y1="60.259" x2="46.0756" y2="61.2394" width="1.016" layer="1"/>
+<wire x1="46.0756" y1="61.2394" x2="46.0756" y2="67.8942" width="1.016" layer="1"/>
+<wire x1="46.0756" y1="67.8942" x2="46.0883" y2="67.9069" width="1.016" layer="1"/>
 </signal>
 <signal name="PROG">
@@
 <contactref element="JP4" pad="9"/>
 <wire x1="34.23" y1="30.17" x2="29.647" y2="30.17" width="0.3" layer="1"/>
-<wire x1="29.647" y1="30.17" x2="28.5623" y2="31.2547" width="0.3" layer="1"/>
-<wire x1="28.5623" y1="31.2547" x2="28.5369" y2="31.2293" width="0.3" layer="1"/>
-<via x="28.5369" y="31.2293" extent="1-16" drill="0.9"/>
-<wire x1="28.5369" y1="31.2293" x2="28.5369" y2="25.9969" width="0.3" layer="16"/>
-<wire x1="28.5369" y1="25.9969" x2="25.4508" y2="22.9108" width="0.3" layer="16"/>
+<wire x1="29.647" y1="30.17" x2="28.63215" y2="31.18485" width="0.3" layer="1"/>
+<wire x1="28.63215" y1="31.18485" x2="28.6893" y2="31.242" width="0.3" layer="1"/>
+<via x="28.6893" y="31.242" extent="1-16" drill="0.9"/>
+<wire x1="28.6893" y1="31.242" x2="28.6893" y2="26.1493" width="0.3" layer="16"/>
+<wire x1="28.6893" y1="26.1493" x2="25.4508" y2="22.9108" width="0.3" layer="16"/>
 <wire x1="25.4508" y1="22.9108" x2="13.1191" y2="22.9108" width="0.3" layer="16"/>
 <wire x1="13.1191" y1="22.9108" x2="9.3091" y2="26.7208" width="0.3" layer="16"/>
@@
 <wire x1="19.05" y1="34.8996" x2="19.05" y2="30.48" width="0.3" layer="16"/>
 <wire x1="26.6954" y1="26.2128" x2="26.6954" y2="30.4292" width="0.3" layer="16"/>
-<wire x1="26.6954" y1="30.4292" x2="26.0731" y2="31.0515" width="0.3" layer="16"/>
-<wire x1="26.0731" y1="31.0515" x2="26.0477" y2="31.0515" width="0.3" layer="16"/>
-<via x="26.0477" y="31.0515" extent="1-16" drill="0.9"/>
-<wire x1="34.23" y1="29.67" x2="27.4292" y2="29.67" width="0.3" layer="1"/>
-<wire x1="27.4292" y1="29.67" x2="26.0477" y2="31.0515" width="0.3" layer="1"/>
+<wire x1="26.6954" y1="30.4292" x2="26.0985" y2="31.0261" width="0.3" layer="16"/>
+<wire x1="26.0985" y1="31.0261" x2="25.8953" y2="31.0261" width="0.3" layer="16"/>
+<via x="25.8953" y="31.0261" extent="1-16" drill="0.9"/>
+<wire x1="34.23" y1="29.67" x2="27.2514" y2="29.67" width="0.3" layer="1"/>
+<wire x1="27.2514" y1="29.67" x2="25.8953" y2="31.0261" width="0.3" layer="1"/>
 <wire x1="21.8313" y1="27.6987" x2="21.8313" y2="25.6159" width="0.3" layer="16"/>
 <wire x1="21.8313" y1="25.6159" x2="23.1775" y2="24.2697" width="0.3" layer="16"/>

Commit message: pcb almost done
Routing:
- net VDD: track 281.8 -> 279.5 mm
Changed lines of the file:
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@@
 <wire x1="53.025" y1="35.3543" x2="53.0098" y2="35.3695" width="0.3" layer="1"/>
 <via x="53.0098" y="35.3695" extent="1-16" drill="1"/>
-<wire x1="53.0098" y1="35.3695" x2="56.3753" y2="35.3695" width="1.016" layer="16"/>
-<wire x1="56.3753" y1="35.3695" x2="62.7507" y2="41.7449" width="1.016" layer="16"/>
-<via x="62.7507" y="41.7449" extent="1-16" drill="1"/>
-<wire x1="62.7507" y1="41.7449" x2="59.878" y2="44.6176" width="1.016" layer="1"/>
-<wire x1="59.878" y1="44.6176" x2="59.878" y2="55.499" width="1.016" layer="1"/>
+<wire x1="53.0098" y1="35.3695" x2="54.7751" y2="35.3695" width="1.016" layer="16"/>
+<wire x1="54.7751" y1="35.3695" x2="63.9064" y2="44.5008" width="1.016" layer="16"/>
+<via x="63.9064" y="44.5008" extent="1-16" drill="1"/>
+<wire x1="63.9064" y1="44.5008" x2="59.878" y2="48.5292" width="1.016" layer="1"/>
+<wire x1="59.878" y1="48.5292" x2="59.878" y2="55.499" width="1.016" layer="1"/>
 <wire x1="95.25" y1="23.18" x2="95.25" y2="40.64" width="1.016" layer="1"/>
 <wire x1="95.25" y1="40.64" x2="91.3384" y2="44.5516" width="1.016" layer="1"/>
@@
 <via x="69.3293" y="44.3992" extent="1-16" drill="1"/>
 <wire x1="69.3293" y1="44.3992" x2="69.3293" y2="44.45" width="0.3" layer="16"/>
-<wire x1="69.3293" y1="44.45" x2="65.4558" y2="44.45" width="1.016" layer="16"/>
-<wire x1="65.4558" y1="44.45" x2="62.7507" y2="41.7449" width="1.016" layer="16"/>
+<wire x1="69.3293" y1="44.45" x2="63.9572" y2="44.45" width="1.016" layer="16"/>
+<wire x1="63.9572" y1="44.45" x2="63.9064" y2="44.5008" width="1.016" layer="16"/>
 <wire x1="42.91" y1="34.35" x2="42.91" y2="27.67" width="0.3" layer="1"/>
 <wire x1="34.23" y1="31.67" x2="33.1" y2="31.67" width="0.3" layer="1"/>
@@
 <wire x1="74.8538" y1="56.2102" x2="74.7903" y2="56.2737" width="0.3" layer="1"/>
 <via x="74.7903" y="56.2737" extent="1-16" drill="1"/>
-<wire x1="74.7903" y1="56.2737" x2="74.7903" y2="57.3786" width="0.8128" layer="16"/>
-<wire x1="74.7903" y1="57.3786" x2="69.6341" y2="62.5348" width="0.8128" layer="16"/>
-<via x="69.6341" y="62.5348" extent="1-16" drill="1"/>
-<wire x1="68.3641" y1="63.8048" x2="69.6341" y2="62.5348" width="1.016" layer="1"/>
-<wire x1="68.3641" y1="63.8048" x2="63.5" y2="63.8048" width="1.016" layer="1"/>
+<wire x1="74.7903" y1="56.2737" x2="74.7903" y2="57.3913" width="0.8128" layer="16"/>
+<wire x1="74.7903" y1="57.3913" x2="69.5325" y2="62.6491" width="0.8128" layer="16"/>
+<via x="69.5325" y="62.6491" extent="1-16" drill="1"/>
+<wire x1="68.3768" y1="63.8048" x2="69.5325" y2="62.6491" width="1.016" layer="1"/>
+<wire x1="68.3768" y1="63.8048" x2="63.5" y2="63.8048" width="1.016" layer="1"/>
 <wire x1="63.5" y1="63.8048" x2="63.1825" y2="63.8048" width="1.016" layer="1"/>
 <wire x1="51.5817" y1="63.9883" x2="63.9699" y2="63.9883" width="1.016" layer="1"/>
-<wire x1="51.5817" y1="63.9883" x2="49.871" y2="65.699" width="1.016" layer="1"/>
+<wire x1="51.5817" y1="63.9883" x2="48.5883" y2="66.9817" width="1.016" layer="1"/>
 <wire x1="63.9699" y1="63.9883" x2="63.9699" y2="65.1383" width="1.016" layer="1"/>
 <wire x1="63.9699" y1="65.1383" x2="65.7098" y2="66.8782" width="1.016" layer="1"/>
 <wire x1="63.9699" y1="63.9883" x2="63.7864" y2="63.8048" width="0.3" layer="1"/>
 <wire x1="63.7864" y1="63.8048" x2="63.5" y2="63.8048" width="0.3" layer="1"/>
-<wire x1="49.871" y1="65.699" x2="48.5883" y2="66.9817" width="1.016" layer="1"/>
 <wire x1="48.5883" y1="66.9817" x2="48.5883" y2="67.9069" width="1.016" layer="1"/>
 </signal>

Commit message: pcb completed
Routing:
- net VDD: track 279.5 -> 281.8 mm
- net GND: track 310.9 -> 309.6 mm
- net +5V: track 39.0 -> 38.4 mm
- added copper zone on layer 1, net BTN_0
- added copper zone on layer 1, net BTN_1
- added copper zone on layer 1, net BTN_2
- added copper zone on layer 1, net BTN_3
- added copper zone on layer 1, net BTN_4
- added copper zone on layer 1, net BTN_COM
- added copper zone on layer 1, net DMMY_0
- added copper zone on layer 1, net N$7
- added copper zone on layer 1, net VBAT+
